Commit message: 更新rf2o参数.

File: src/robot_description/urdf/robot_gazebo.urdf (robot description, URDF)
Before this commit: robot robot, 7 links, 6 joints
Links:
- removed link behind_boll_link
- link base_link: geometry collision box size=0.12 0.08 0.10; collision box size=0.16 0.20 0.10
- link left_wheel_link: geometry collision cylinder length=0.025 radius=0.035; visual cylinder length=0.025 radius=0.035
- link right_wheel_link: geometry collision cylinder length=0.025 radius=0.035; visual cylinder length=0.025 radius=0.035
Joints:
- removed joint behind_boll_joint
- joint front_boll_joint: origin xyz=0.025 0 -0.015 -> xyz=0.18 0 -0.015
- joint imu_joint: origin xyz=0 0 0.03 rpy=0 0 0 -> xyz=0 0 0 rpy=0 0 0
- joint laser_joint: origin xyz=0 0 0.03 rpy=0 0 0 -> xyz=0.10 0 0.285 rpy=0 0 0
- joint left_wheel_joint: origin xyz=0 0.05 -0.015 rpy=1.57079 0 0 -> xyz=0 0.15 0.0 rpy=1.57079 0 0
- joint right_wheel_joint: origin xyz=0 -0.05 -0.015 rpy=1.57079 0 0 -> xyz=0 -0.15 0.0 rpy=1.57079 0 0

Commit message: Sync car real robot workspace

File: src/robot_description/urdf/robot_gazebo.urdf (robot description, URDF)
Before this commit: robot robot, 6 links, 5 joints
Links:
- removed link front_boll_link
- removed link left_wheel_link
- removed link right_wheel_link
- added link base_footprint
- added link caster_wheel; collision sphere radius=0.015; visual sphere radius=0.015
- added link left_wheel, mass 0.15; collision cylinder length=0.03 radius=0.05; visual cylinder length=0.03 radius=0.05
- added link right_wheel, mass 0.15; collision cylinder length=0.03 radius=0.05; visual cylinder length=0.03 radius=0.05
- link base_link: mass 0.2 -> 2.0; geometry collision box size=0.25 0.22 0.10; visual box size=0.25 0.22 0.10
Joints:
- removed joint front_boll_joint
- added joint base_joint: type fixed, parent base_footprint, child base_link, origin xyz=0 0 0.05 rpy=0 0 0
- added joint caster_wheel_joint: type fixed, parent base_link, child caster_wheel, origin xyz=-0.12 0 -0.035 rpy=0 0 0
- joint imu_joint: origin xyz=0 0 0 rpy=0 0 0 -> xyz=-0.1357881 0.0051315 0.0907072 rpy=3.1415926535897931 0 -1.5707963267948966
- joint laser_joint: origin xyz=0.10 0 0.285 rpy=0 0 0 -> xyz=0 0 0.15 rpy=0 0 0
- joint left_wheel_joint: axis 0 0 -1 -> 0 0 1; child left_wheel_link -> left_wheel; origin xyz=0 0.15 0.0 rpy=1.57079 0 0 -> xyz=0 0.1474 0 rpy=-1.5707963267948966 0 0
- joint right_wheel_joint: axis 0 0 -1 -> 0 0 1; child right_wheel_link -> right_wheel; origin xyz=0 -0.15 0.0 rpy=1.57079 0 0 -> xyz=0 -0.1474 0 rpy=-1.5707963267948966 0 0

Commit message: set imu joint rotation to zero

File: src/robot_description/urdf/robot_gazebo.urdf (robot description, URDF)
Before this commit: robot robot, 7 links, 6 joints
Joints:
- joint imu_joint: origin xyz=-0.1357881 0.0051315 0.0907072 rpy=0 0 -1.5707963267948966 -> xyz=-0.1357881 0.0051315 0.0907072 rpy=0 0 0
