Commit message: Fix IMU frame rotation in robot description

File: src/differential_drive.urdf.xacro (robot description, xacro)
@@ -23,7 +23,11 @@
     wheel_mid=(100, 0, -124.72)mm
     imu-base = (-135.7881, 5.1315, 90.7072)mm
-    IMU frame orientation matches the sensor mounting:
-    yaw=-90deg plus roll=180deg, so sensor_z points opposite base_link_z.
-    This corresponds to imu_cartographer_publisher axis_map=-y,-x,-z.
+    IMU frame orientation matches the current sensor mounting:
+    only yaw=-90deg relative to base_link.
+    坐标变换关系为：
+    x_base =  y_imu
+    y_base = -x_imu
+    z_base =  z_imu
+    因此对应 imu_cartographer_publisher 的 axis_map=y,-x,z。
   -->
   <xacro:property name="imu_x" value="-0.1357881"/>
@@ -200,5 +204,5 @@
     <parent link="base_link"/>
     <child link="imu_link"/>
-    <origin xyz="${imu_x} ${imu_y} ${imu_z}" rpy="${M_PI} 0 -${M_PI/2}"/>
+    <origin xyz="${imu_x} ${imu_y} ${imu_z}" rpy="0 0 -${M_PI/2}"/>
   </joint>
   <link name="imu_link"/>

File: src/robot_description/urdf/robot_gazebo.urdf (robot description, URDF)
Before this commit: robot robot, 7 links, 6 joints
Joints:
- joint imu_joint: origin xyz=-0.1357881 0.0051315 0.0907072 rpy=3.1415926535897931 0 -1.5707963267948966 -> xyz=-0.1357881 0.0051315 0.0907072 rpy=0 0 -1.5707963267948966

Commit message: Adjust IMU yaw alignment for odom orientation

File: src/differential_drive.urdf.xacro (robot description, xacro)
@@ -24,10 +24,10 @@
     imu-base = (-135.7881, 5.1315, 90.7072)mm
     IMU frame orientation matches the current sensor mounting:
-    only yaw=-90deg relative to base_link.
+    only yaw=+90deg relative to base_link.
     坐标变换关系为：
-    x_base =  y_imu
-    y_base = -x_imu
+    x_base = -y_imu
+    y_base =  x_imu
     z_base =  z_imu
-    因此对应 imu_cartographer_publisher 的 axis_map=y,-x,z。
+    因此对应 imu_cartographer_publisher 的 axis_map=-y,x,z。
   -->
   <xacro:property name="imu_x" value="-0.1357881"/>
@@ -204,5 +204,5 @@
     <parent link="base_link"/>
     <child link="imu_link"/>
-    <origin xyz="${imu_x} ${imu_y} ${imu_z}" rpy="0 0 -${M_PI/2}"/>
+    <origin xyz="${imu_x} ${imu_y} ${imu_z}" rpy="0 0 ${M_PI/2}"/>
   </joint>
   <link name="imu_link"/>

File: src/robot_description/urdf/robot_gazebo.urdf (robot description, URDF)
Before this commit: robot robot, 7 links, 6 joints
Joints:
- joint imu_joint: origin xyz=-0.1357881 0.0051315 0.0907072 rpy=0 0 -1.5707963267948966 -> xyz=-0.1357881 0.0051315 0.0907072 rpy=0 0 1.5707963267948966

Commit message: Align imu_link orientation with base_link

File: src/differential_drive.urdf.xacro (robot description, xacro)
@@ -23,11 +23,10 @@
     wheel_mid=(100, 0, -124.72)mm
     imu-base = (-135.7881, 5.1315, 90.7072)mm
-    IMU frame orientation matches the current sensor mounting:
-    only yaw=+90deg relative to base_link.
-    坐标变换关系为：
-    x_base = -y_imu
-    y_base =  x_imu
-    z_base =  z_imu
-    因此对应 imu_cartographer_publisher 的 axis_map=-y,x,z。
+    当前将 imu_link 直接对齐到 base_link，
+    即两者姿态完全一致，满足：
+    x_base = x_imu
+    y_base = y_imu
+    z_base = z_imu
+    因此对应 imu_cartographer_publisher 的 axis_map=x,y,z。
   -->
   <xacro:property name="imu_x" value="-0.1357881"/>
@@ -204,5 +203,5 @@
     <parent link="base_link"/>
     <child link="imu_link"/>
-    <origin xyz="${imu_x} ${imu_y} ${imu_z}" rpy="0 0 ${M_PI/2}"/>
+    <origin xyz="${imu_x} ${imu_y} ${imu_z}" rpy="0 0 0"/>
   </joint>
   <link name="imu_link"/>

File: src/robot_description/urdf/robot_gazebo.urdf (robot description, URDF)
Before this commit: robot robot, 7 links, 6 joints
Joints:
- joint imu_joint: origin xyz=-0.1357881 0.0051315 0.0907072 rpy=0 0 1.5707963267948966 -> xyz=-0.1357881 0.0051315 0.0907072 rpy=0 0 0

Commit message: Restore inverted IMU mounting configuration

File: src/differential_drive.urdf.xacro (robot description, xacro)
@@ -23,10 +23,12 @@
     wheel_mid=(100, 0, -124.72)mm
     imu-base = (-135.7881, 5.1315, 90.7072)mm
-    当前将 imu_link 直接对齐到 base_link，
-    即两者姿态完全一致，满足：
-    x_base = x_imu
-    y_base = y_imu
-    z_base = z_imu
-    因此对应 imu_cartographer_publisher 的 axis_map=x,y,z。
+    IMU 实体为倒装安装，并且相对 base_link 还绕 z 轴旋转了 -90deg。
+    因此 imu_link 相对 base_link 的旋转取：
+    R = Rz(-pi/2) * Rx(pi)
+    对应坐标轴关系为：
+    x_base = -y_imu
+    y_base = -x_imu
+    z_base = -z_imu
+    因此对应 imu_cartographer_publisher 的 axis_map=-y,-x,-z。
   -->
   <xacro:property name="imu_x" value="-0.1357881"/>
@@ -203,5 +205,5 @@
     <parent link="base_link"/>
     <child link="imu_link"/>
-    <origin xyz="${imu_x} ${imu_y} ${imu_z}" rpy="0 0 0"/>
+    <origin xyz="${imu_x} ${imu_y} ${imu_z}" rpy="${M_PI} 0 -${M_PI/2}"/>
   </joint>
   <link name="imu_link"/>

File: src/robot_description/urdf/robot_gazebo.urdf (robot description, URDF)
Before this commit: robot robot, 7 links, 6 joints
Joints:
- joint imu_joint: origin xyz=-0.1357881 0.0051315 0.0907072 rpy=0 0 0 -> xyz=-0.1357881 0.0051315 0.0907072 rpy=3.1415926535897931 0 -1.5707963267948966

Commit message: Add wheel speed feedback odometry

File: src/differential_drive.urdf.xacro (robot description, xacro)
@@ -9,5 +9,5 @@
   <xacro:property name="base_height" value="0.1"/>
   <!-- 轮子参数 -->
-  <xacro:property name="wheel_radius" value="0.05"/>  <!-- 直径10cm，半径5cm -->
+  <xacro:property name="wheel_radius" value="0.0175"/>  <!-- 直径3.5cm，半径1.75cm -->
   <xacro:property name="wheel_width" value="0.03"/>
   <xacro:property name="wheel_mass" value="0.15"/>

File: src/robot_description/urdf/robot_gazebo.urdf (robot description, URDF)
Before this commit: robot robot, 7 links, 6 joints
Links:
- link left_wheel: geometry collision cylinder length=0.03 radius=0.0175; visual cylinder length=0.03 radius=0.0175
- link right_wheel: geometry collision cylinder length=0.03 radius=0.0175; visual cylinder length=0.03 radius=0.0175
Joints:
- joint base_joint: origin xyz=0 0 0.05 rpy=0 0 0 -> xyz=0 0 0.0175 rpy=0 0 0
- joint caster_wheel_joint: origin xyz=-0.12 0 -0.035 rpy=0 0 0 -> xyz=-0.12 0 -0.0025 rpy=0 0 0

Commit message: Raise robot base link model height

File: src/differential_drive.urdf.xacro (robot description, xacro)
@@ -8,4 +8,5 @@
   <xacro:property name="base_width" value="0.22"/>
   <xacro:property name="base_height" value="0.1"/>
+  <xacro:property name="base_link_height" value="${base_height/2}"/>  <!-- base_link 位于车体中心，高于地面 5cm -->
   <!-- 轮子参数 -->
   <xacro:property name="wheel_radius" value="0.0175"/>  <!-- 直径3.5cm，半径1.75cm -->
@@ -19,5 +20,5 @@
   <!--
     IMU measured offset in base_link frame (meter).
-    Derived from shell-center measurements with wheel-midpoint as base_link proxy:
+    Derived from shell-center measurements with wheel-midpoint as the original base_link proxy:
     imu=(-35.7881, 5.1315, -34.0128)mm
     wheel_mid=(100, 0, -124.72)mm
@@ -90,5 +91,5 @@
     <parent link="base_footprint"/>
     <child link="base_link"/>
-    <origin xyz="0 0 ${wheel_radius}" rpy="0 0 0"/>
+    <origin xyz="0 0 ${base_link_height}" rpy="0 0 0"/>
   </joint>
   <link name="base_link">
@@ -112,5 +113,5 @@
     <parent link="base_link"/>
     <child link="left_wheel"/>
-    <origin xyz="0 ${track_width/2} 0" rpy="${-M_PI/2} 0 0"/>
+    <origin xyz="0 ${track_width/2} ${wheel_radius-base_link_height}" rpy="${-M_PI/2} 0 0"/>
     <axis xyz="0 0 1"/>
   </joint>
@@ -135,5 +136,5 @@
     <parent link="base_link"/>
     <child link="right_wheel"/>
-    <origin xyz="0 ${-track_width/2} 0" rpy="${-M_PI/2} 0 0"/>
+    <origin xyz="0 ${-track_width/2} ${wheel_radius-base_link_height}" rpy="${-M_PI/2} 0 0"/>
     <axis xyz="0 0 1"/>
   </joint>
@@ -158,5 +159,5 @@
     <parent link="base_link"/>
     <child link="caster_wheel"/>
-    <origin xyz="${caster_x} 0 ${-wheel_radius+caster_radius}" rpy="0 0 0"/>
+    <origin xyz="${caster_x} 0 ${caster_radius-base_link_height}" rpy="0 0 0"/>
   </joint>
   <link name="caster_wheel">
@@ -180,5 +181,5 @@
     <parent link="base_link"/>
     <child link="laser_link"/>
-    <origin xyz="0 0 ${laser_height-wheel_radius}" rpy="0 0 0"/>
+    <origin xyz="0 0 ${laser_height-base_link_height}" rpy="0 0 0"/>
   </joint>
   <link name="laser_link">
@@ -205,5 +206,5 @@
     <parent link="base_link"/>
     <child link="imu_link"/>
-    <origin xyz="${imu_x} ${imu_y} ${imu_z}" rpy="${M_PI} 0 -${M_PI/2}"/>
+    <origin xyz="${imu_x} ${imu_y} ${wheel_radius+imu_z-base_link_height}" rpy="${M_PI} 0 -${M_PI/2}"/>
   </joint>
   <link name="imu_link"/>

File: src/robot_description/urdf/robot_gazebo.urdf (robot description, URDF)
Before this commit: robot robot, 7 links, 6 joints
Joints:
- joint base_joint: origin xyz=0 0 0.0175 rpy=0 0 0 -> xyz=0 0 0.05 rpy=0 0 0
- joint caster_wheel_joint: origin xyz=-0.12 0 -0.0025 rpy=0 0 0 -> xyz=-0.12 0 -0.035 rpy=0 0 0
- joint imu_joint: origin xyz=-0.1357881 0.0051315 0.0907072 rpy=0 0 0 -> xyz=-0.1357881 0.0051315 0.0582072 rpy=0 0 0
- joint left_wheel_joint: origin xyz=0 0.1474 0 rpy=-1.5707963267948966 0 0 -> xyz=0 0.1474 -0.0325 rpy=-1.5707963267948966 0 0
- joint right_wheel_joint: origin xyz=0 -0.1474 0 rpy=-1.5707963267948966 0 0 -> xyz=0 -0.1474 -0.0325 rpy=-1.5707963267948966 0 0

Commit message: 修改电机速度方向.

File: src/differential_drive.urdf.xacro (robot description, xacro)
@@ -181,5 +181,5 @@
     <parent link="base_link"/>
     <child link="laser_link"/>
-    <origin xyz="0 0 ${laser_height-base_link_height}" rpy="0 0 0"/>
+    <origin xyz="0 0 ${laser_height-base_link_height}" rpy="0 0 ${M_PI}"/>
   </joint>
   <link name="laser_link">

File: src/robot_description/urdf/robot_gazebo.urdf (robot description, URDF)
Before this commit: robot robot, 7 links, 6 joints
Joints:
- joint laser_joint: origin xyz=0 0 0.15 rpy=0 0 0 -> xyz=0 0 0.15 rpy=0 0 3.141592653589793

Commit message: 修改整车朝向.

File: src/differential_drive.urdf.xacro (robot description, xacro)
@@ -181,5 +181,5 @@
     <parent link="base_link"/>
     <child link="laser_link"/>
-    <origin xyz="0 0 ${laser_height-base_link_height}" rpy="0 0 ${M_PI}"/>
+    <origin xyz="0 0 ${laser_height-base_link_height}" rpy="0 0 0"/>
   </joint>
   <link name="laser_link">

File: src/robot_description/urdf/robot_gazebo.urdf (robot description, URDF)
Before this commit: robot robot, 7 links, 6 joints
Joints:
- joint laser_joint: origin xyz=0 0 0.15 rpy=0 0 3.141592653589793 -> xyz=0 0 0.15 rpy=0 0 0

Commit message: Disable raw odom input and update wheel config

File: src/differential_drive.urdf.xacro (robot description, xacro)
@@ -10,5 +10,5 @@
   <xacro:property name="base_link_height" value="${base_height/2}"/>  <!-- base_link 位于车体中心，高于地面 5cm -->
   <!-- 轮子参数 -->
-  <xacro:property name="wheel_radius" value="0.0175"/>  <!-- 直径3.5cm，半径1.75cm -->
+  <xacro:property name="wheel_radius" value="0.035"/>  <!-- 直径7cm，半径3.5cm -->
   <xacro:property name="wheel_width" value="0.03"/>
   <xacro:property name="wheel_mass" value="0.15"/>

File: src/robot_description/urdf/robot_gazebo.urdf (robot description, URDF)
Before this commit: robot robot, 7 links, 6 joints
Links:
- link left_wheel: geometry collision cylinder length=0.03 radius=0.035; visual cylinder length=0.03 radius=0.035
- link right_wheel: geometry collision cylinder length=0.03 radius=0.035; visual cylinder length=0.03 radius=0.035
